File: schematics/BotController/BotController.sch (KiCad schematic (older format))
At the start: 20 parts, among them IC1 ATMEGA644-P, SW2 reset, X1 CRYSTAL_OSSCI

Commit message: Schulter revised
Parts:
- gave numbers to parts that had none: 9
Changed lines of the file:
@@
 MISO
 $Comp
-L +5V #PWR01
+L +5V #PWR1
 U 1 1 50E5D5BA
 P 5050 1700
-F 0 "#PWR01" H 5050 1790 20  0001 C CNN
+F 0 "#PWR1" H 5050 1790 20  0001 C CNN
 F 1 "+5V" H 5050 1790 30  0000 C CNN
 F 2 "" H 5050 1700 60  0001 C CNN
@@
 SCK
 $Comp
-L +5V #PWR02
+L +5V #PWR2
 U 1 1 57173265
 P 5050 1700
-F 0 "#PWR02" H 5050 1790 20  0001 C CNN
+F 0 "#PWR2" H 5050 1790 20  0001 C CNN
 F 1 "+5V" H 5050 1790 30  0000 C CNN
 F 2 "" H 5050 1700 60  0001 C CNN
@@
 $EndComp
 $Comp
-L CONN_01X03 P?
+L CONN_01X03 P1
 U 1 1 571B9A9C
 P 6250 6750
-F 0 "P?" H 6250 6950 50  0000 C CNN
+F 0 "P1" H 6250 6950 50  0000 C CNN
 F 1 "UM2102 - UART2USB" V 6350 6750 50  0000 C CNN
 F 2 "" H 6250 6750 60  0000 C CNN
@@
 GND
 $Comp
-L LED D?
+L LED D2
 U 1 1 57251F35
 P 7050 2050
-F 0 "D?" H 7050 2150 50  0000 C CNN
+F 0 "D2" H 7050 2150 50  0000 C CNN
 F 1 "LED" H 7050 1950 50  0000 C CNN
 F 2 "" H 7050 2050 60  0000 C CNN
@@
 Connection ~ 3700 3500
 $Comp
-L POT RV?
+L POT RV1
 U 1 1 572524E5
 P 3700 4750
-F 0 "RV?" H 3700 4650 50  0000 C CNN
+F 0 "RV1" H 3700 4650 50  0000 C CNN
 F 1 "10K" H 3700 4750 50  0000 C CNN
 F 2 "" H 3700 4750 60  0000 C CNN
@@
 	6100 2400 6050 2400
 $Comp
-L CONN_01X04 P?
+L CONN_01X04 P2
 U 1 1 57261EF0
 P 7200 6750
-F 0 "P?" H 7200 7000 50  0000 C CNN
+F 0 "P2" H 7200 7000 50  0000 C CNN
 F 1 "Herkulex Servo" V 7300 6750 50  0000 C CNN
 F 2 "" H 7200 6750 60  0000 C CNN
@@
 	9400 6200 9400 4300
 $Comp
-L R R?
+L R R3
 U 1 1 5727190E
 P 8950 3800
-F 0 "R?" V 9030 3800 50  0000 C CNN
+F 0 "R3" V 9030 3800 50  0000 C CNN
 F 1 "1.5K" V 8950 3800 50  0000 C CNN
 F 2 "" V 8880 3800 30  0000 C CNN
@@
 $EndComp
 $Comp
-L R R?
+L R R4
 U 1 1 57271C02
 P 9150 3800
-F 0 "R?" V 9230 3800 50  0000 C CNN
+F 0 "R4" V 9230 3800 50  0000 C CNN
 F 1 "1.5K" V 9150 3800 50  0000 C CNN
 F 2 "" V 9080 3800 30  0000 C CNN
@@
 	9150 3650 9150 1700
 $Comp
-L CONN_01X04 P?
+L CONN_01X04 P4
 U 1 1 572B216F
 P 9600 4150
-F 0 "P?" H 9600 4400 50  0000 C CNN
+F 0 "P4" H 9600 4400 50  0000 C CNN
 F 1 "Encoder Socket" V 9700 4150 50  0000 C CNN
 F 2 "" H 9600 4150 60  0000 C CNN
@@
 ConflictEncoderGND
 $Comp
-L CONN_01X04 P?
+L CONN_01X04 P3
 U 1 1 572B75C3
 P 8700 3050
-F 0 "P?" H 8700 3300 50  0000 C CNN
+F 0 "P3" H 8700 3300 50  0000 C CNN
 F 1 "Encoder Socket 0" V 8800 3050 50  0000 C CNN
 F 2 "" H 8700 3050 60  0000 C CNN
@@
 Connection ~ 8300 4100
 $Comp
-L CONN_01X04 P?
+L CONN_01X04 P5
 U 1 1 572E5E87
 P 10100 2550
-F 0 "P?" H 10100 2800 50  0000 C CNN
+F 0 "P5" H 10100 2800 50  0000 C CNN
 F 1 "Stepper 1 WristTurn" V 10200 2550 50  0000 C CNN
 F 2 "" H 10100 2550 60  0000 C CNN

Commit message: no message
Parts:
- added C1: 100uF, symbol CP
- added C2: 100nF, symbol C
- added P10: Stepper Upperarm, symbol CONN_01X04
- added P11: Stepper Shoulder, symbol CONN_01X04
- added P6: POWER uC, symbol CONN_01X02
- added P7: POWER_SERVO, symbol CONN_01X02
- added P8: Stepper Ellbow, symbol CONN_01X04
- added P9: Stepper Forearm, symbol CONN_01X04
- added U1: 7805, symbol 7805
Connections:
- net RST is gone; now on net EN2: AVR1.5, C15.1, D1.1 (A), IC1.9 (~RESET), R1.2, SW2.2
- net +5V: now also U1.VO; no longer P2.2 (P2)
- net CLK1: now also P5.3 (P3); no longer P5.2 (P2)
- net DIR1: now also P5.2 (P2); no longer P5.3 (P3)
- net En5: now reaches IC1.18 ((PCINT28/OC1B)PD4)
- net En5: now also P11.1 (P1)
- net CLK5: now reaches IC1.19 ((PCINT294/OC1A)PD5)
- net CLK5: now also P11.3 (P3)
- net DIR5: now reaches IC1.20 ((PCINT30/OC2B/ICP)PD6)
- net DIR5: now also P11.2 (P2)
- net EN4: now reaches IC1.21 ((PCINT31/OC2A)PD7)
- net EN4: now also P10.1 (P1)
- net CLK4: now reaches IC1.24 ((PCINT18/TCK)PC2)
- net CLK4: now also P10.3 (P3)
- net DIR4: now reaches IC1.25 ((PCINT19/TMS)PC3)
- net DIR4: now also P10.2 (P2)
- net EN3: now reaches IC1.26 ((PCINT20/TDO)PC4)
- net EN3: now also P9.1 (P1)
- net CLK3: now reaches IC1.27 ((PCINT21/TDI)PC5)
- net CLK3: now also P9.3 (P3)
- net DIR2: now reaches IC1.28 ((PCINT22/TOSC1)PC6)
- net DIR2: now also IC1.34 ((PCINT6/ADC6)PA6), P8.2 (P2), P9.2 (P2)
- net EN2: now reaches IC1.29 ((PCINT23/TOSC2)PC7)
- net EN2: now also P8.1 (P1)
- net CLK2: now reaches IC1.33 ((PCINT7/ADC7)PA7)
- net CLK2: now also P8.3 (P3)
- net GND renamed GNDPWR
- net GNDPWR: now also C1.2, C2.2, P10.4 (P4), P11.4 (P4), P6.2 (P2), P7.2 (P2), P8.4 (P4), P9.4 (P4), U1.GND
- new net: P2.2 (P2), P7.1 (P1)
- new net: C1.1, C2.1, P6.1 (P1), U1.VI
- no-connect marks 23 -> 8
Other:
- moved on the sheet: P3
